File: Electronics/tripteron/tripteron.kicad_sch (KiCad schematic)
At the start: 27 parts, among them J1 Conn_01x02_Pin, J2 Conn_01x04_Pin, J3 Conn_01x04_Pin, J4 Conn_01x04_Pin, J5 Conn_01x04_Pin, J6 Conn_01x04_Pin

Commit message: uncertanty and V2 boards
Parts:
- removed A1, A3, A4, A5, A6: Pololu_Breakout_A4988, Module:Pololu_Breakout-16_15.2x20.3mm, symbol Driver_Motor:Pololu_Breakout_A4988
- removed A2: RaspberryPi_Pico, Module:RaspberryPi_Pico_Common_THT, symbol MCU_Module:RaspberryPi_Pico
- removed J1: Conn_01x02_Pin, Connector_PinSocket_2.54mm:PinSocket_1x02_P2.54mm_Vertical, symbol Connector:Conn_01x02_Pin
- removed J2, J3, J4, J5, J6: Conn_01x04_Pin, Connector_PinHeader_2.54mm:PinHeader_1x04_P2.54mm_Vertical, symbol Connector:Conn_01x04_Pin
- removed TP1, TP10, TP11, TP12, TP13, TP14, TP15, TP2, TP3, TP4, TP5, TP6, TP7, TP8, TP9: TestPoint, TestPoint:TestPoint_Pad_2.5x2.5mm, symbol Connector:TestPoint
- added A1: Arduino_Nano_RP2040_Connect, Module:Arduino_Nano, symbol MCU_Module:Arduino_Nano_RP2040_Connect
- added C1, C2: C, Capacitor_SMD:C_0603_1608Metric_Pad1.08x0.95mm_HandSolder, symbol Device:C
- added D1, D2, D3: LED, Capacitor_SMD:C_0603_1608Metric_Pad1.08x0.95mm_HandSolder, symbol Device:LED
- added H1, H2: MountingHole_Pad, MountingHole:MountingHole_3.2mm_M3_DIN965_Pad, symbol Mechanical:MountingHole_Pad
- added J1, J3, J8: Conn_01x03_Pin, Connector_PinHeader_2.54mm:PinHeader_1x03_P2.54mm_Vertical, symbol Connector:Conn_01x03_Pin
- added J2, J5, J6, J7: Conn_01x02_Pin, Connector_PinHeader_2.54mm:PinHeader_1x02_P2.54mm_Vertical, symbol Connector:Conn_01x02_Pin
- added J4: Conn_01x10_Pin, Connector_PinHeader_2.54mm:PinHeader_1x10_P2.54mm_Vertical, symbol Connector:Conn_01x10_Pin
- added JP1: SolderJumper_2_Open, Jumper:SolderJumper-2_P1.3mm_Open_RoundedPad1.0x1.5mm, symbol Jumper:SolderJumper_2_Open
- added R1, R2, R3: R, Resistor_SMD:R_0603_1608Metric_Pad0.98x0.95mm_HandSolder, symbol Device:R
- added U1: NCP1117-3.3_SOT223, Package_TO_SOT_SMD:SOT-223-3_TabPin2, symbol Regulator_Linear:NCP1117-3.3_SOT223
Connections:
- net GND: now also A1.29 (GND), A1.4 (GND), C1.2, C2.2, H1.1, H2.1, J4.1 (Pin_1), J4.2 (Pin_2), J4.3 (Pin_3), J4.4 (Pin_4), J4.5 (Pin_5), R1.2, R2.2, R3.2, U1.1 (GND)
- new net: D2.1 (K), R2.1
- new net: D3.1 (K), R3.1
- new net: A1.21 (A2), D3.2 (A)
- new net: D1.1 (K), R1.1
- new net: A1.19 (A0), D1.2 (A)
- new net: A1.20 (A1), D2.2 (A)
- new net: A1.17 (3V3), JP1.1 (A)
- new net 3.3V: C2.1, J4.10 (Pin_10), J4.6 (Pin_6), J4.7 (Pin_7), J4.8 (Pin_8), J4.9 (Pin_9), JP1.2 (B), U1.2 (VO)
- new net GPIO_1: A1.22 (A3), J8.3 (Pin_3)
- new net GPIO_2: A1.25 (A6), J8.2 (Pin_2)
- new net GPIO_3: A1.26 (A7), J8.1 (Pin_1)
- new net INT_1: A1.14 (D11/COPI), J3.3 (Pin_3)
- new net INT_2: A1.15 (D12/CIPO), J3.2 (Pin_2)
- new net INT_3: A1.16 (D13/SCK), J3.1 (Pin_1)
- new net M1_DIR: A1.5 (D2), J2.2 (Pin_2)
- new net M1_STP: A1.6 (D3), J2.1 (Pin_1)
- new net M2_DIR: A1.7 (D4), J5.2 (Pin_2)
- new net M2_STP: A1.8 (D5), J5.1 (Pin_1)
- new net M3_DIR: A1.9 (D6), J7.2 (Pin_2)
- new net M3_STP: A1.10 (D7), J7.1 (Pin_1)
- new net SCL: A1.24 (SCL/A5), J6.1 (Pin_1)
- new net SDA: A1.23 (SDA/A4), J6.2 (Pin_2)
- new net VUSB: A1.27 (VUSB/5V), C1.1, U1.3 (VI)
- new net XSHUT_1: A1.11 (D8), J1.3 (Pin_3)
- new net XSHUT_2: A1.12 (D9), J1.2 (Pin_2)
- new net XSHUT_3: A1.13 (D10/CS), J1.1 (Pin_1)
- no-connect marks 9 -> 0
Other:
- note added: "3.3V LDO to reduce load on arduino ldo this allows upto 1A and is powered from VUSB if not used, solder jumper to use arduinos 3.3 reg"
- note added: "MAY REQUIRE LEVEL SHIFTING, CHECK BEFORE ORDERING"
- note removed: "8-35V DC"
- note removed: "SPEC: SUPPORT FOR 5 MOTOR DRIVERS 12/24V INPUT @ 10A MAX DECOUPLING ON MOTOR PSU 5/3V LOGIC FOR ESP AND DRIVERS MICRO SWITCHES FOR MICROSTEP ADJUSTMENT STEPPER DRIVERS ARE 8X2 2.54MM WITH 12.5MM SPACING"
